File: kicad-flex-sensor/_autosave-kicad-flex-sensor.kicad_sch (KiCad schematic)
At the start: 8 parts, among them J1 Power, J2 Digital/PWM, J3 Analog, J4 Digital/PWM

Commit message: add plein de choses
Parts:
- added C1, C2, C3, C4: C, symbol Device:C
- added R1, R2, R3, R4, R5: R, symbol Device:R
Connections:
- new net: C1.1, R1.1, R2.1, R5.2
- new net: C3.2, R5.1
Other:
- moved on the sheet: U4
