File: kicad-flex-sensor/_autosave-kicad-flex-sensor.kicad_pcb (KiCad board)
At the start: 2 copper layers, 68.6 x 53.3 mm, 11 parts, among them J1 Power, J2 Digital/PWM, J3 Analog, J4 Digital/PWM

Commit message: add plein de choses
Parts:
- added U4: ~, Package_DIP:DIP-8_W7.62mm_LongPads, F.Cu at (114.3, 76.1)
- moved U1 7.41 mm to (128.8, 58.7)
- moved U2 5.49 mm to (138.5, 80.7)

Commit message: Routage
Parts:
- added C1: 100n, Capacitor_THT:C_Disc_D4.7mm_W2.5mm_P5.00mm, F.Cu at (139.4, 86.6)
- added C2: 100n, Capacitor_THT:C_Disc_D4.7mm_W2.5mm_P5.00mm, F.Cu at (139.4, 90.6)
- added C4: 1u, Capacitor_THT:C_Rect_L7.0mm_W4.5mm_P5.00mm, F.Cu at (139.4, 80.9)
- added R1: 100k, Resistor_THT:R_Axial_DIN0207_L6.3mm_D2.5mm_P7.62mm_Horizontal, F.Cu at (120.6, 69.2)
- added R2: 1k, Resistor_THT:R_Axial_DIN0207_L6.3mm_D2.5mm_P7.62mm_Horizontal, F.Cu at (120.6, 73.2)
- added R3: 100k, Resistor_THT:R_Axial_DIN0207_L6.3mm_D2.5mm_P7.62mm_Horizontal, F.Cu at (120.6, 77.3)
- added R4: 1k, Resistor_THT:R_Axial_DIN0207_L6.3mm_D2.5mm_P7.62mm_Horizontal, F.Cu at (120.6, 81.3)
- added R5: 10k, Resistor_THT:R_Axial_DIN0207_L6.3mm_D2.5mm_P7.62mm_Horizontal, F.Cu at (120.6, 85.4)
- added U5: LTC1050CN8, graphite_empreinte:PDIP-8_N, F.Cu at (141.5, 74.6)
- added U6: ~, graphite_empreinte:Capteur, F.Cu at (110.4, 78.0)
- moved U1 30.0 mm to (158.8, 58.7), turned to 90 degrees
- moved U2 22.9 mm to (157.9, 92.8), turned to 180 degrees
- moved U3 22.6 mm to (137.7, 55.1), turned to 0 degrees
- moved U4 21.0 mm to (113.6, 55.1)
Connections:
- J2 pad 5: /13 -> D13
- J2 pad 7: /*11 -> D11
- J2 pad 8: /*10 -> D10
- J3 pad 1: /A0 -> A0
- J3 pad 5: /SDA/A4 -> A4
- J3 pad 6: /SCL/A5 -> A5
- J4 pad 3: /*5 -> D5
- J4 pad 4: /4 -> D4
- J4 pad 6: /2 -> D2
- J4 pad 7: /TX/1 -> D1
- J4 pad 8: /RX/0 -> D0
- U1 pad 1: unconnected-(U1-Vcc-Pad1) -> +5V
- U1 pad 2: unconnected-(U1-GND-Pad2) -> GND
- U1 pad 3: unconnected-(U1-TxD-Pad3) -> D0
- U1 pad 4: unconnected-(U1-RxD-Pad4) -> D1
- U2 pad 1: unconnected-(U2-GND-Pad1) -> GND
- U2 pad 2: unconnected-(U2-VCC-Pad2) -> +5V
- U2 pad 3: unconnected-(U2-SCL-Pad3) -> A5
- U2 pad 4: unconnected-(U2-SDA-Pad4) -> A4
- U3 pad 1: unconnected-(U3-GND-Pad1) -> GND
- U3 pad 2: unconnected-(U3-VCC-Pad2) -> +5V
- U3 pad 3: unconnected-(U3-SW-Pad3) -> D5
- U3 pad 4: unconnected-(U3-DT-Pad4) -> D4
- U3 pad 5: unconnected-(U3-CLK-Pad5) -> D2
- U4 pad 1: unconnected-(U4-SS-Pad1) -> D10
- U4 pad 2: unconnected-(U4-SCK-Pad2) -> D13
- U4 pad 3: unconnected-(U4-MOSI-Pad3) -> D11
- U4 pad 4: unconnected-(U4-GND-Pad4) -> GND
- U4 pad 5: unconnected-(U4-VCC-Pad5) -> +5V
- U4 pad 7: unconnected-(U4-GND-Pad7) -> GND
- U4 pad 8: unconnected-(U4-VCC-Pad8) -> +5V
Routing:
- net GND: track 0.00 -> 177.1 mm
- net +5V: track 0.00 -> 169.9 mm
- net A0: track 0.00 -> 72.9 mm
- net Net-(U5-V+): track 0.00 -> 49.9 mm
- net Net-(U5-OUT): track 0.00 -> 45.0 mm
- net Net-(U5-V-): track 0.00 -> 34.9 mm
- net D10: track 0.00 -> 29.6 mm
- net D13: track 0.00 -> 21.4 mm
- net D2: track 0.00 -> 18.3 mm
- net D5: track 0.00 -> 15.7 mm
- net D4: track 0.00 -> 15.7 mm
- net Net-(U6-C-): track 0.00 -> 12.0 mm
- net A4: track 0.00 -> 11.2 mm
- net D0: track 0.00 -> 10.2 mm
- net A5: track 0.00 -> 8.99 mm
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- added copper zone on B.Cu, net D11
- removed copper zone on B.Cu, net GND
