File: kicad-flex-sensor/kicad-flex-sensor.kicad_pcb (KiCad board)
At the start: 2 copper layers, 68.6 x 53.3 mm, 11 parts, among them J1 Power, J2 Digital/PWM, J3 Analog, J4 Digital/PWM

Commit message: Routage
Parts:
- added C1: 100n, Capacitor_THT:C_Disc_D4.7mm_W2.5mm_P5.00mm, F.Cu at (139.4, 86.6)
- added C2: 100n, Capacitor_THT:C_Disc_D4.7mm_W2.5mm_P5.00mm, F.Cu at (139.4, 90.6)
- added C4: 1u, Capacitor_THT:C_Rect_L7.0mm_W4.5mm_P5.00mm, F.Cu at (139.4, 80.9)
- added R1: 100k, Resistor_THT:R_Axial_DIN0207_L6.3mm_D2.5mm_P7.62mm_Horizontal, F.Cu at (120.6, 69.2)
- added R2: 1k, Resistor_THT:R_Axial_DIN0207_L6.3mm_D2.5mm_P7.62mm_Horizontal, F.Cu at (120.6, 73.2)
- added R3: 100k, Resistor_THT:R_Axial_DIN0207_L6.3mm_D2.5mm_P7.62mm_Horizontal, F.Cu at (120.6, 77.3)
- added R4: 1k, Resistor_THT:R_Axial_DIN0207_L6.3mm_D2.5mm_P7.62mm_Horizontal, F.Cu at (120.6, 81.3)
- added R5: 10k, Resistor_THT:R_Axial_DIN0207_L6.3mm_D2.5mm_P7.62mm_Horizontal, F.Cu at (120.6, 85.4)
- added U4: ~, Package_DIP:DIP-8_W7.62mm_LongPads, F.Cu at (128.3, 54.4)
- added U5: LTC1050CN8, graphite_empreinte:PDIP-8_N, F.Cu at (141.5, 74.6)
- added U6: ~, graphite_empreinte:Capteur, F.Cu at (110.4, 78.0)
- moved U2 27.9 mm to (157.9, 92.8), turned to 180 degrees
- moved U1 22.8 mm to (158.3, 64.5), turned to 90 degrees
- moved U3 16.0 mm to (151.3, 53.6), turned to 0 degrees
Connections:
- J1 pad 5: +5V -> D11
- J1 pad 6: GND -> D11
- J1 pad 7: GND -> D11
- J2 pad 4: GND -> D11
- J2 pad 5: /13 -> D13
- J2 pad 7: /*11 -> D11
- J2 pad 8: /*10 -> D10
- J3 pad 1: /A0 -> A0
- J3 pad 5: /SDA/A4 -> A4
- J3 pad 6: /SCL/A5 -> A5
- J4 pad 3: /*5 -> D5
- J4 pad 4: /4 -> D4
- J4 pad 6: /2 -> D2
- J4 pad 7: /TX/1 -> D1
- J4 pad 8: /RX/0 -> D0
- U1 pad 1: unconnected-(U1-Vcc-Pad1) -> D11
- U1 pad 2: unconnected-(U1-GND-Pad2) -> D11
- U1 pad 3: unconnected-(U1-TxD-Pad3) -> D0
- U1 pad 4: unconnected-(U1-RxD-Pad4) -> D1
- U2 pad 1: unconnected-(U2-GND-Pad1) -> D11
- U2 pad 2: unconnected-(U2-VCC-Pad2) -> D11
- U2 pad 3: unconnected-(U2-SCL-Pad3) -> A5
- U2 pad 4: unconnected-(U2-SDA-Pad4) -> A4
- U3 pad 1: unconnected-(U3-GND-Pad1) -> D11
- U3 pad 2: unconnected-(U3-VCC-Pad2) -> D11
- U3 pad 3: unconnected-(U3-SW-Pad3) -> D5
- U3 pad 4: unconnected-(U3-DT-Pad4) -> D4
- U3 pad 5: unconnected-(U3-CLK-Pad5) -> D2
Routing:
- net Net-(U5-OUT): track 0.00 -> 56.6 mm
- net Net-(U5-V+): track 0.00 -> 53.1 mm
- net Net-(U5-V-): track 0.00 -> 35.1 mm
- net A0: track 0.00 -> 29.3 mm
- net D0: track 0.00 -> 16.2 mm
- net D1: track 0.00 -> 12.6 mm
- net Net-(U6-C-): track 0.00 -> 12.0 mm
- net D10: track 0.00 -> 10.7 mm
- net D13: track 0.00 -> 9.28 mm
- net A5: track 0.00 -> 8.99 mm
- net A4: track 0.00 -> 8.98 mm
- net D2: track 0.00 -> 6.02 mm
- net D5: track 0.00 -> 4.61 mm
- net D4: track 0.00 -> 4.61 mm
- added copper zone on B.Cu, net D11
- removed copper zone on B.Cu, net GND

Commit message: Les trucs que j'avais pas  sauvegardé
Parts:
- moved U4 14.7 mm to (113.6, 55.1)
- moved U3 13.6 mm to (137.7, 55.1)
- moved U1 5.78 mm to (158.8, 58.7)
Connections:
- C1 pad 2: D11 -> GND
- C2 pad 2: D11 -> GND
- J1 pad 5: D11 -> +5V
- J1 pad 6: D11 -> GND
- J1 pad 7: D11 -> GND
- J2 pad 4: D11 -> GND
- R1 pad 2: D11 -> GND
- R2 pad 2: D11 -> GND
- U1 pad 1: D11 -> +5V
- U1 pad 2: D11 -> GND
- U2 pad 1: D11 -> GND
- U2 pad 2: D11 -> +5V
- U3 pad 1: D11 -> GND
- U3 pad 2: D11 -> +5V
- U4 pad 4: D11 -> GND
- U4 pad 5: D11 -> +5V
- U4 pad 7: D11 -> GND
- U4 pad 8: D11 -> +5V
- U5 pad 2: D11 -> GND
- U5 pad 3: D11 -> +5V
- U6 pad 1: D11 -> +5V
Routing:
- net GND: track 0.00 -> 183.1 mm
- net +5V: track 0.00 -> 165.9 mm
- net D10: track 10.7 -> 29.6 mm
- net Net-(U5-V+): track 53.1 -> 68.1 mm
- net D5: track 4.61 -> 17.7 mm
- net D2: track 6.02 -> 18.3 mm
- net D13: track 9.28 -> 21.4 mm
- net D4: track 4.61 -> 15.7 mm
- net Net-(U5-OUT): track 56.6 -> 45.6 mm
- net Net-(U5-V-): track 35.1 -> 25.5 mm
- net D0: track 16.2 -> 10.2 mm
- net D1: track 12.6 -> 6.59 mm
- net A0: track 29.3 -> 34.5 mm

Commit message: routage qui marche !
Parts:
- moved C1 26.1 mm to (113.8, 91.6)
- moved R2 22.2 mm to (142.0, 67.4), turned to 90 degrees
- moved AOP1 19.9 mm to (125.1, 85.8), turned to 180 degrees
- moved R4 19.5 mm to (139.0, 74.8), turned to -90 degrees
- moved R1 19.3 mm to (113.5, 87.1)
- moved R5 15.3 mm to (105.5, 83.1)
- moved Screen1 11.7 mm to (153.9, 81.8), turned to 90 degrees
- moved Encodeur1 11.7 mm to (128.9, 62.7), turned to -90 degrees
- moved C4 8.65 mm to (131.9, 76.6), turned to 180 degrees
- moved R3 6.29 mm to (125.3, 81.5)
- moved Potar1 5.90 mm to (117.4, 59.6), turned to -90 degrees
- moved Capteur1 3.70 mm to (107.2, 76.1)
- moved Bluetooth1 1.95 mm to (157.9, 57.0), turned to 180 degrees
- moved C2 1.95 mm to (139.8, 88.7)
- renumbered U5 to AOP1, U1 to Bluetooth1, U6 to Capteur1, U3 to Encodeur1, U4 to Potar1, U2 to Screen1
Connections:
- J3 pad 2: /A1 -> A1
- Potar1 pad 5: +5V -> GND
- Potar1 pad 6: unconnected-(U4-P0W-Pad6) -> GND
- Potar1 pad 7: GND -> A1
Routing:
- net GND: track 183.1 -> 0.00 mm
- net A5: track 8.99 -> 73.6 mm
- net Net-(AOP1-V+): track 68.1 -> 23.1 mm
- net +5V: track 165.9 -> 128.5 mm
- net D11: track 0.00 -> 31.3 mm
- net D2: track 18.3 -> 37.2 mm
- net Net-(AOP1-OUT): track 45.6 -> 26.9 mm
- net D4: track 15.7 -> 31.1 mm
- net A4: track 8.98 -> 22.9 mm
- net D5: track 17.7 -> 29.9 mm
- net A0: track 34.5 -> 22.6 mm
- net D10: track 29.6 -> 23.5 mm
- net D1: track 6.59 -> 10.7 mm
- net Net-(Capteur1-C-): track 12.0 -> 8.23 mm
- net Net-(AOP1-V-): track 25.5 -> 28.7 mm
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- added copper zone on B.Cu, net GND
- removed copper zone on B.Cu, net D11

Commit message: Finito !
Parts:
- removed R2: 1k, Resistor_THT:R_Axial_DIN0207_L6.3mm_D2.5mm_P7.62mm_Horizontal
- added FlexSensor1: ~, graphite_empreinte:Capteur, F.Cu at (151.6, 91.3)
- added R6: 47k, Resistor_THT:R_Axial_DIN0207_L6.3mm_D2.5mm_P7.62mm_Horizontal, F.Cu at (157.1, 93.0)
- moved R4 10.4 mm to (129.1, 77.9), turned to 0 degrees
- moved Screen1 7.02 mm to (157.6, 75.8)
- moved C4 3.20 mm to (131.9, 73.4)
Connections:
- J3 pad 2: A1 -> /A1
- J3 pad 3: /A2 -> A2
- Potar1 pad 7: A1 -> Net-(AOP1-V-)
Routing:
- net A5: track 73.6 -> 30.5 mm, vias 0 -> 2
- net +5V: track 128.5 -> 143.8 mm
- net A2: track 0.00 -> 9.72 mm
- net Net-(AOP1-OUT): track 26.9 -> 19.0 mm
- net A0: track 22.6 -> 26.8 mm
- net A4: track 22.9 -> 27.0 mm
- net Net-(AOP1-V-): track 28.7 -> 32.5 mm
- net D5: track 29.9 -> 27.5 mm
- net Net-(AOP1-V+): track 23.1 -> 21.2 mm
