File: kicad-flex-sensor/kicad-flex-sensor.kicad_sch (KiCad schematic)
At the start: 8 parts, among them J1 Power, J2 Digital/PWM, J3 Analog, J4 Digital/PWM

Commit message: Routage
Parts:
- added C1, C2: 100n, Capacitor_THT:C_Disc_D4.7mm_W2.5mm_P5.00mm, symbol Device:C
- added C4: 1u, Capacitor_THT:C_Rect_L7.0mm_W4.5mm_P5.00mm, symbol Device:C
- added R1, R3: 100k, Resistor_THT:R_Axial_DIN0207_L6.3mm_D2.5mm_P7.62mm_Horizontal, symbol Device:R
- added R2, R4: 1k, Resistor_THT:R_Axial_DIN0207_L6.3mm_D2.5mm_P7.62mm_Horizontal, symbol Device:R
- added R5: 10k, Resistor_THT:R_Axial_DIN0207_L6.3mm_D2.5mm_P7.62mm_Horizontal, symbol Device:R
- added U5: LTC1050CN8, graphite_empreinte:PDIP-8_N, symbol Graphite_symbol:LTC1050CN8
- added U6: ~, graphite_empreinte:Capteur, symbol Graphite_symbol:Capteur
Connections:
- net *10 is gone; now on net D10: J2.8 (Pin_8)
- net *11 is gone; now on net D11: J2.7 (Pin_7)
- net *5 is gone; now on net D5: J4.3 (Pin_3)
- net 13 is gone; now on net D13: J2.5 (Pin_5)
- net 2 is gone; now on net D2: J4.6 (Pin_6)
- net 4 is gone; now on net D4: J4.4 (Pin_4)
- net RX/0 is gone; now on net D0: J4.8 (Pin_8)
- net SCL/A5 is gone; now on net A5: J3.6 (Pin_6)
- net SDA/A4 is gone; now on net A4: J3.5 (Pin_5)
- net TX/1 is gone; now on net D1: J4.7 (Pin_7)
- net +5V: now also U1.1 (Vcc), U2.2 (VCC), U3.2 (VCC), U4.5 (VCC), U4.8 (VCC), U5.3 (+IN), U6.1 (C+)
- net A0: now also C2.1, R4.2
- net GND: now also U1.2 (GND), U2.1 (GND), U3.1 (GND), U4.4 (GND), U4.7 (GND), C1.2, C2.2, R1.2, R2.2, U5.2 (-IN)
- net D0: now reaches U1.3 (TxD)
- net D1: now reaches U1.4 (RxD)
- net A5: now reaches U2.3 (SCL)
- net A4: now reaches U2.4 (SDA)
- net D5: now reaches U3.3 (SW)
- net D4: now reaches U3.4 (DT)
- net D2: now reaches U3.5 (CLK)
- net D10: now reaches U4.1 (SS)
- net D13: now reaches U4.2 (SCK)
- net D11: now reaches U4.3 (MOSI)
- new net: C4.1, R2.1, R3.2, U5.4 (V-)
- new net: C4.2, R3.1, R4.1, U5.6 (OUT)
- new net: R5.1, U6.2 (C-)
- new net: C1.1, R1.1, R5.2, U5.7 (V+)
Other:
- moved on the sheet: U4

Commit message: routage qui marche !
Parts:
- renumbered U5 to AOP1, U1 to Bluetooth1, U6 to Capteur1, U3 to Encodeur1, U4 to Potar1, U2 to Screen1
Connections:
- net +5V: no longer Potar1.5 (VCC)
- net A1: now also Potar1.7 (P0B)
- net GND: now also Potar1.5 (P0A), Potar1.6 (P0W); no longer Potar1.7 (GND)
Changed lines of the file:
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@@
 	)
 	(junction
-		(at 116.84 91.44)
-		(diameter 0)
-		(color 0 0 0 0)
-	)
-	(junction
 		(at 31.75 46.99)
 		(diameter 1.016)
@@
 	)
 	(junction
+		(at 86.36 95.25)
+		(diameter 0)
+		(color 0 0 0 0)
+	)
+	(junction
 		(at 219.71 111.76)
 		(diameter 0)
@@
 	)
 	(junction
-		(at 86.36 95.25)
+		(at 114.3 91.44)
 		(diameter 0)
 		(color 0 0 0 0)
@@
 	(wire
 		(pts
-			(xy 114.3 95.25) (xy 86.36 95.25)
-		)
-		(stroke
-			(width 0)
-			(type default)
-		)
-	)
-	(wire
-		(pts
 			(xy 86.36 33.02) (xy 86.36 53.34)
 		)
@@
 	(wire
 		(pts
-			(xy 116.84 91.44) (xy 116.84 96.52)
+			(xy 113.03 88.9) (xy 114.3 88.9)
+		)
+		(stroke
+			(width 0)
+			(type default)
+		)
+	)
+	(wire
+		(pts
+			(xy 123.19 83.82) (xy 123.19 96.52)
 		)
 		(stroke
@@
 	(wire
 		(pts
-			(xy 116.84 83.82) (xy 116.84 91.44)
-		)
-		(stroke
-			(width 0)
-			(type default)
-		)
-	)
-	(wire
-		(pts
 			(xy 88.9 50.8) (xy 92.71 50.8)
 		)
@@
 	(wire
 		(pts
-			(xy 86.36 95.25) (xy 86.36 96.52)
+			(xy 86.36 91.44) (xy 86.36 95.25)
 		)
 		(stroke
@@
 	(wire
 		(pts
-			(xy 86.36 91.44) (xy 86.36 95.25)
+			(xy 86.36 95.25) (xy 86.36 96.52)
 		)
 		(stroke
@@
 	(wire
 		(pts
-			(xy 113.03 83.82) (xy 116.84 83.82)
-		)
-		(stroke
-			(width 0)
-			(type default)
-		)
-	)
-	(wire
-		(pts
 			(xy 219.71 106.68) (xy 219.71 111.76)
 		)
@@
 	(wire
 		(pts
+			(xy 114.3 91.44) (xy 114.3 95.25)
+		)
+		(stroke
+			(width 0)
+			(type default)
+		)
+	)
+	(wire
+		(pts
 			(xy 62.23 34.29) (xy 64.77 34.29)
 		)
@@
 	(wire
 		(pts
+			(xy 114.3 95.25) (xy 86.36 95.25)
+		)
+		(stroke
+			(width 0)
+			(type default)
+		)
+	)
+	(wire
+		(pts
 			(xy 116.84 132.08) (xy 125.73 132.08)
 		)
@@
 	(wire
 		(pts
+			(xy 114.3 88.9) (xy 114.3 91.44)
+		)
+		(stroke
+			(width 0)
+			(type default)
+		)
+	)
+	(wire
+		(pts
 			(xy 219.71 111.76) (xy 231.14 111.76)
 		)
@@
 	(wire
 		(pts
-			(xy 114.3 86.36) (xy 114.3 95.25)
+			(xy 113.03 83.82) (xy 123.19 83.82)
 		)
 		(stroke
@@
 	(wire
 		(pts
-			(xy 113.03 91.44) (xy 116.84 91.44)
-		)
-		(stroke
-			(width 0)
-			(type default)
-		)
-	)
-	(wire
-		(pts
 			(xy 80.01 86.36) (xy 92.71 86.36)
 		)
@@
 	(wire
 		(pts
-			(xy 116.84 96.52) (xy 88.9 96.52)
+			(xy 123.19 96.52) (xy 88.9 96.52)
 		)
 		(stroke
@@
 	(wire
 		(pts
+			(xy 113.03 91.44) (xy 114.3 91.44)
+		)
+		(stroke
+			(width 0)
+			(type default)
+		)
+	)
+	(wire
+		(pts
 			(xy 62.23 49.53) (xy 74.93 49.53)
 		)
@@
 		)
 	)
+	(global_label "A1"
+		(shape passive)
+		(at 114.3 86.36 0)
+		(fields_autoplaced yes)
+		(effects
+			(font
+				(size 1.27 1.27)
+			)
+			(justify left)
+		)
+		(property "Intersheetrefs" "${INTERSHEET_REFS}"
+			(at 118.6624 86.36 0)
+			(effects
+				(font
+					(size 1.27 1.27)
+				)
+				(justify left)
+				(hide yes)
+			)
+		)
+	)
 	(global_label "D10"
 		(shape passive)
@@
 		)
 	)
+	(global_label "A1"
+		(shape passive)
+		(at 21.59 62.23 180)
+		(fields_autoplaced yes)
+		(effects
+			(font
+				(size 1.27 1.27)
+			)
+			(justify right)
+		)
+		(property "Intersheetrefs" "${INTERSHEET_REFS}"
+			(at 17.2276 62.23 0)
+			(effects
+				(font
+					(size 1.27 1.27)
+				)
+				(justify right)
+				(hide yes)
+			)
+		)
+	)
 	(global_label "A0"
 		(shape passive)
@@
 		(dnp no)
 		(fields_autoplaced yes)
-		(property "Reference" "U1"
+		(property "Reference" "Bluetooth1"
 			(at 116.84 53.9749 0)
 			(effects
@@
 			(project ""
 				(path "/e63e39d7-6ac0-4ffd-8aa3-1841a4541b55"
-					(reference "U1")
+					(reference "Bluetooth1")
 					(unit 1)
 				)
@@
 		(dnp no)
 		(fields_autoplaced yes)
-		(property "Reference" "U6"
+		(property "Reference" "Capteur1"
 			(at 82.55 99.06 0)
 			(effects
@@
 			(project ""
 				(path "/e63e39d7-6ac0-4ffd-8aa3-1841a4541b55"
-					(reference "U6")
+					(reference "Capteur1")
 					(unit 1)
 				)
@@
 		(dnp no)
 		(fields_autoplaced yes)
-		(property "Reference" "U5"
+		(property "Reference" "AOP1"
 			(at 171.45 92.71 0)
 			(effects
@@
 			(project ""
 				(path "/e63e39d7-6ac0-4ffd-8aa3-1841a4541b55"
-					(reference "U5")
+					(reference "AOP1")
 					(unit 1)
 				)
@@
 		(dnp no)
 		(fields_autoplaced yes)
-		(property "Reference" "U2"
+		(property "Reference" "Screen1"
 			(at 114.3 69.8499 0)
 			(effects
@@
 			(project ""
 				(path "/e63e39d7-6ac0-4ffd-8aa3-1841a4541b55"
-					(reference "U2")
+					(reference "Screen1")
 					(unit 1)
 				)
@@
 		(dnp no)
 		(fields_autoplaced yes)
-		(property "Reference" "U3"
+		(property "Reference" "Encodeur1"
 			(at 111.76 36.8299 0)
 			(effects
@@
 			(project ""
 				(path "/e63e39d7-6ac0-4ffd-8aa3-1841a4541b55"
-					(reference "U3")
+					(reference "Encodeur1")
 					(unit 1)
 				)
@@
 		(dnp no)
 		(fields_autoplaced yes)
-		(property "Reference" "U4"
+		(property "Reference" "Potar1"
 			(at 102.87 76.2 0)
 			(effects
@@
 			(project ""
 				(path "/e63e39d7-6ac0-4ffd-8aa3-1841a4541b55"
-					(reference "U4")
+					(reference "Potar1")
 					(unit 1)
 				)

Commit message: Finito !
Parts:
- removed R2: 1k, Resistor_THT:R_Axial_DIN0207_L6.3mm_D2.5mm_P7.62mm_Horizontal, symbol Device:R
- added FlexSensor1: ~, graphite_empreinte:Capteur, symbol Graphite_symbol:FlexSensor
- added R6: 47k, Resistor_THT:R_Axial_DIN0207_L6.3mm_D2.5mm_P7.62mm_Horizontal, symbol Device:R
Connections:
- net +5V: now also FlexSensor1.1 (Vcc)
- net A1: no longer Potar1.7 (P0B)
- net A2: now also FlexSensor1.2 (GND), R6.1
- net GND: now also R6.2
- net at AOP1.4 (V-), C4.1, R3.2: now also Potar1.7 (P0B)
