File: 2. Kicad/kicad-flex-sensor/kicad-flex-sensor.kicad_sch (KiCad schematic)
At the start: 19 parts, among them J1 Power, J2 Digital/PWM, J3 Analog, J4 Digital/PWM

Commit message: Organisation du github - kicad
Connections:
- net +5V: now also AOP1.7 (V+); no longer AOP1.3 (+IN)
- net GND: now also AOP1.4 (V-); no longer AOP1.2 (-IN)
- net at C4.1, Potar1.7 (P0B), R3.2: now also AOP1.2 (-IN); no longer AOP1.4 (V-)
- net at C1.1, R1.1, R5.2: now also AOP1.3 (+IN); no longer AOP1.7 (V+)
Changed lines of the file:
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@@
+	)
+	(junction
+		(at 116.84 113.03)
+		(diameter 0)
+		(color 0 0 0 0)
 	)
 	(junction
@@
 	)
 	(junction
-		(at 133.35 110.49)
-		(diameter 0)
-		(color 0 0 0 0)
-	)
-	(junction
-		(at 116.84 113.03)
-		(diameter 0)
-		(color 0 0 0 0)
-	)
-	(junction
 		(at 140.97 132.08)
 		(diameter 0)
@@
 	)
 	(junction
+		(at 137.16 93.98)
+		(diameter 0)
+		(color 0 0 0 0)
+	)
+	(junction
 		(at 114.3 91.44)
 		(diameter 0)
@@
 	)
 	(junction
-		(at 137.16 107.95)
-		(diameter 0)
-		(color 0 0 0 0)
-	)
-	(junction
 		(at 88.9 72.39)
+		(diameter 0)
+		(color 0 0 0 0)
+	)
+	(junction
+		(at 133.35 105.41)
 		(diameter 0)
 		(color 0 0 0 0)
@@
 	(wire
 		(pts
-			(xy 143.51 118.11) (xy 201.93 118.11)
+			(xy 133.35 105.41) (xy 143.51 105.41)
 		)
 		(stroke
@@
 	(wire
 		(pts
-			(xy 113.03 86.36) (xy 119.38 86.36)
+			(xy 113.03 86.36) (xy 118.11 86.36)
 		)
 		(stroke
@@
 	(wire
 		(pts
-			(xy 201.93 105.41) (xy 199.39 105.41)
-		)
-		(stroke
-			(width 0)
-			(type default)
-		)
-	)
-	(wire
-		(pts
 			(xy 62.23 26.67) (xy 74.93 26.67)
 		)
@@
 	(wire
 		(pts
-			(xy 201.93 118.11) (xy 201.93 105.41)
-		)
-		(stroke
-			(width 0)
-			(type default)
-		)
-	)
-	(wire
-		(pts
 			(xy 31.75 46.99) (xy 31.75 52.07)
 		)
@@
 	(wire
 		(pts
+			(xy 199.39 105.41) (xy 203.2 105.41)
+		)
+		(stroke
+			(width 0)
+			(type default)
+		)
+	)
+	(wire
+		(pts
 			(xy 86.36 74.93) (xy 92.71 74.93)
 		)
@@
 	(wire
 		(pts
-			(xy 140.97 105.41) (xy 140.97 132.08)
+			(xy 140.97 110.49) (xy 140.97 132.08)
 		)
 		(stroke
@@
 	(wire
 		(pts
-			(xy 133.35 110.49) (xy 133.35 88.9)
-		)
-		(stroke
-			(width 0)
-			(type default)
-		)
-	)
-	(wire
-		(pts
 			(xy 31.75 26.67) (xy 31.75 39.37)
 		)
@@
 	(wire
 		(pts
-			(xy 143.51 105.41) (xy 140.97 105.41)
-		)
-		(stroke
-			(width 0)
-			(type default)
-		)
-	)
-	(wire
-		(pts
 			(xy 62.23 62.23) (xy 74.93 62.23)
 		)
@@
 	(wire
 		(pts
-			(xy 119.38 86.36) (xy 119.38 110.49)
+			(xy 118.11 86.36) (xy 118.11 105.41)
+		)
+		(stroke
+			(width 0)
+			(type default)
+		)
+	)
+	(wire
+		(pts
+			(xy 203.2 105.41) (xy 203.2 93.98)
+		)
+		(stroke
+			(width 0)
+			(type default)
+		)
+	)
+	(wire
+		(pts
+			(xy 138.43 107.95) (xy 138.43 113.03)
 		)
 		(stroke
@@
 	(wire
 		(pts
-			(xy 137.16 107.95) (xy 143.51 107.95)
-		)
-		(stroke
-			(width 0)
-			(type default)
-		)
-	)
-	(wire
-		(pts
 			(xy 86.36 33.02) (xy 92.71 33.02)
 		)
@@
 	(wire
 		(pts
+			(xy 137.16 93.98) (xy 203.2 93.98)
+		)
+		(stroke
+			(width 0)
+			(type default)
+		)
+	)
+	(wire
+		(pts
 			(xy 125.73 113.03) (xy 125.73 118.11)
 		)
@@
 	(wire
 		(pts
-			(xy 125.73 113.03) (xy 143.51 113.03)
-		)
-		(stroke
-			(width 0)
-			(type default)
-		)
-	)
-	(wire
-		(pts
-			(xy 143.51 113.03) (xy 143.51 118.11)
-		)
-		(stroke
-			(width 0)
-			(type default)
-		)
-	)
-	(wire
-		(pts
 			(xy 133.35 88.9) (xy 208.28 88.9)
 		)
@@
 	(wire
 		(pts
+			(xy 133.35 105.41) (xy 133.35 88.9)
+		)
+		(stroke
+			(width 0)
+			(type default)
+		)
+	)
+	(wire
+		(pts
 			(xy 208.28 88.9) (xy 208.28 99.06)
 		)
@@
 	(wire
 		(pts
+			(xy 143.51 107.95) (xy 138.43 107.95)
+		)
+		(stroke
+			(width 0)
+			(type default)
+		)
+	)
+	(wire
+		(pts
 			(xy 88.9 35.56) (xy 88.9 24.13)
 		)
@@
 	(wire
 		(pts
+			(xy 138.43 113.03) (xy 125.73 113.03)
+		)
+		(stroke
+			(width 0)
+			(type default)
+		)
+	)
+	(wire
+		(pts
 			(xy 92.71 113.03) (xy 97.79 113.03)
 		)
@@
 	(wire
 		(pts
-			(xy 119.38 110.49) (xy 133.35 110.49)
+			(xy 140.97 110.49) (xy 143.51 110.49)
+		)
+		(stroke
+			(width 0)
+			(type default)
+		)
+	)
+	(wire
+		(pts
+			(xy 118.11 105.41) (xy 133.35 105.41)
 		)
 		(stroke
@@
 	(wire
 		(pts
+			(xy 137.16 93.98) (xy 137.16 107.95)
+		)
+		(stroke
+			(width 0)
+			(type default)
+		)
+	)
+	(wire
+		(pts
 			(xy 62.23 69.85) (xy 74.93 69.85)
 		)
@@
 	(wire
 		(pts
-			(xy 143.51 110.49) (xy 133.35 110.49)
-		)
-		(stroke
-			(width 0)
-			(type default)
-		)
-	)
-	(wire
-		(pts
 			(xy 62.23 74.93) (xy 74.93 74.93)
 		)
@@
 	(wire
 		(pts
-			(xy 137.16 85.09) (xy 137.16 107.95)
-		)
-		(stroke
+			(xy 137.16 85.09) (xy 137.16 93.98)
+		)
+		(stroke
